File: _autosave-STM32 Dev Board.kicad_pcb (KiCad board)
At the start: 2 copper layers, 38.5 x 32.7 mm, 36 parts, among them J5 2 Pin JST, J6 USB_B_Micro, Q1 PMOS, U1 MCP2221AxML, U2 STM32F070F6Px, U3 MCP1824S, U4 MCP73113

Commit message: generated BOM
Routing:
- net VUSB: track 69.4 -> 56.6 mm
- net Net-(U2-NRST): track 22.8 -> 22.0 mm
- net 3.3V: track 52.8 -> 53.5 mm
Changed lines of the file:
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@@
 	)
 	(via
-		(at 136.2 72.3)
+		(at 136.55 72)
 		(size 0.6)
 		(drill 0.3)
@@
 	)
 	(segment
+		(start 142.7 72)
+		(end 143.35 72.65)
+		(width 0.2)
+		(layer "F.Cu")
+		(net 19)
+	)
+	(segment
 		(start 142.601414 77.8)
 		(end 142.1125 77.8)
@@
 	)
 	(segment
+		(start 143.35 73.55)
+		(end 143.4 73.6)
+		(width 0.2)
+		(layer "F.Cu")
+		(net 19)
+	)
+	(segment
 		(start 142.675 71.975)
 		(end 142.7 72)
@@
 	)
 	(segment
-		(start 142.7 72)
-		(end 142.7 72.9)
-		(width 0.2)
-		(layer "F.Cu")
-		(net 19)
-	)
-	(segment
 		(start 139.2 74.75)
 		(end 138.95 74.5)
@@
 	)
 	(segment
-		(start 142.7 72.9)
-		(end 143.4 73.6)
-		(width 0.2)
-		(layer "F.Cu")
-		(net 19)
-	)
-	(segment
 		(start 143.4 73.6)
 		(end 143.4 77.001414)
@@
 		(net 19)
 	)
+	(segment
+		(start 143.35 72.65)
+		(end 143.35 73.55)
+		(width 0.2)
+		(layer "F.Cu")
+		(net 19)
+	)
 	(via
 		(at 138.95 74.5)
@@
 	)
 	(segment
-		(start 134 67.66)
-		(end 134 67.8)
-		(width 0.2)
-		(layer "B.Cu")
-		(net 19)
-	)
-	(segment
 		(start 148.5375 80.35)
 		(end 149.1 79.7875)
@@
 	)
 	(segment
+		(start 142.3 75.65)
+		(end 142.3 78.25)
+		(width 0.2)
+		(layer "B.Cu")
+		(net 19)
+	)
+	(segment
 		(start 142.7 72)
 		(end 141 73.7)
@@
 	)
 	(segment
-		(start 142.7 75.1)
-		(end 143 75.4)
-		(width 0.2)
-		(layer "B.Cu")
-		(net 19)
-	)
-	(segment
-		(start 142.3 76.1)
-		(end 143 75.4)
-		(width 0.2)
-		(layer "B.Cu")
-		(net 19)
-	)
-	(segment
-		(start 148.55 69)
-		(end 146.3 69)
-		(width 0.2)
-		(layer "B.Cu")
-		(net 19)
-	)
-	(segment
-		(start 146.3 69)
-		(end 135.2 69)
+		(start 144.059 76.491)
+		(end 149.091 76.491)
+		(width 0.2)
+		(layer "B.Cu")
+		(net 19)
+	)
+	(segment
+		(start 134 67.66)
+		(end 134.01 67.66)
+		(width 0.2)
+		(layer "B.Cu")
+		(net 19)
+	)
+	(segment
+		(start 138.35 72)
+		(end 135.2 68.85)
 		(width 0.2)
 		(layer "B.Cu")
@@
 	)
 	(segment
+		(start 135.2 68.85)
+		(end 135.2 69)
+		(width 0.2)
+		(layer "B.Cu")
+		(net 19)
+	)
+	(segment
 		(start 149.1 79.7875)
-		(end 149.1 69.55)
+		(end 149.1 76.5)
 		(width 0.2)
 		(layer "B.Cu")
@@
 	)
 	(segment
-		(start 143 75.4)
-		(end 146.3 72.1)
-		(width 0.2)
-		(layer "B.Cu")
-		(net 19)
-	)
-	(segment
-		(start 142.3 78.25)
-		(end 142.3 76.1)
-		(width 0.2)
-		(layer "B.Cu")
-		(net 19)
-	)
-	(segment
-		(start 146.3 72.1)
-		(end 146.3 69)
+		(start 134.01 67.66)
+		(end 135.2 68.85)
+		(width 0.2)
+		(layer "B.Cu")
+		(net 19)
+	)
+	(segment
+		(start 149.091 76.491)
+		(end 149.1 76.5)
 		(width 0.2)
 		(layer "B.Cu")
@@
 	)
 	(segment
-		(start 134 67.8)
-		(end 135.2 69)
+		(start 142.7 72)
+		(end 142.7 75.25)
+		(width 0.2)
+		(layer "B.Cu")
+		(net 19)
+	)
+	(segment
+		(start 142.3 78.25)
+		(end 144.059 76.491)
 		(width 0.2)
 		(layer "B.Cu")
@@
 	)
 	(segment
-		(start 149.1 69.55)
-		(end 148.55 69)
-		(width 0.2)
-		(layer "B.Cu")
-		(net 19)
-	)
-	(segment
 		(start 141 73.7)
 		(end 140.3 73.7)
@@
 	)
 	(segment
+		(start 142.7 72)
+		(end 138.35 72)
+		(width 0.2)
+		(layer "B.Cu")
+		(net 19)
+	)
+	(segment
 		(start 152.3 75.875)
 		(end 152.8 75.875)
@@
 	)
 	(segment
-		(start 142.7 72)
-		(end 142.7 75.1)
-		(width 0.2)
-		(layer "B.Cu")
-		(net 19)
-	)
-	(segment
 		(start 154.3875 77.4625)
 		(end 155.6 77.4625)
@@
 	)
 	(segment
+		(start 142.7 75.25)
+		(end 142.3 75.65)
+		(width 0.2)
+		(layer "B.Cu")
+		(net 19)
+	)
+	(segment
 		(start 155.6 74.3625)
 		(end 155.6 70.4625)
@@
 	)
 	(segment
+		(start 139.775 81.475)
+		(end 140 81.7)
+		(width 0.2)
+		(layer "F.Cu")
+		(net 30)
+	)
+	(segment
 		(start 140 85.3)
 		(end 139.475 85.825)
@@
 	(segment
 		(start 139.6 81.3)
-		(end 140 81.7)
+		(end 139.775 81.475)
 		(width 0.2)
 		(layer "F.Cu")
@@
 		(net 30)
 	)
-	(via
-		(at 138.8 81.05)
+	(segment
+		(start 139.775 81.475)
+		(end 140.3 80.95)
+		(width 0.2)
+		(layer "F.Cu")
+		(net 30)
+	)
+	(via
+		(at 140.3 80.95)
 		(size 0.6)
 		(drill 0.3)
@@
 	)
 	(segment
-		(start 140 80)
-		(end 138.95 81.05)
+		(start 145.58 80)
+		(end 141.25 80)
 		(width 0.2)
 		(layer "B.Cu")
@@
 	)
 	(segment
-		(start 145.58 80)
-		(end 140 80)
-		(width 0.2)
-		(layer "B.Cu")
-		(net 30)
-	)
-	(segment
-		(start 138.95 81.05)
-		(end 138.8 81.05)
+		(start 141.25 80)
+		(end 140.3 80.95)
 		(width 0.2)
 		(layer "B.Cu")
@@
 		(layer "B.Cu")
 		(net 31)
+	)
+	(segment
+		(start 141.9 86.475)
+		(end 141.9 79.9)
+		(width 0.2)
+		(layer "F.Cu")
+		(net 32)
 	)
 	(segment
@@
 	)
 	(segment
-		(start 141.85 81.3)
-		(end 141.85 86.425)
-		(width 0.2)
-		(layer "F.Cu")
-		(net 32)
-	)
-	(segment
 		(start 135.9625 79.1625)
 		(end 135.625 79.1625)
-		(width 0.2)
-		(layer "F.Cu")
-		(net 32)
-	)
-	(segment
-		(start 141.85 86.425)
-		(end 141.9 86.475)
 		(width 0.2)
 		(layer "F.Cu")
@@
 	)
 	(segment
-		(start 141.85 79.95)
-		(end 145 76.8)
-		(width 0.2)
-		(layer "F.Cu")
-		(net 32)
-	)
-	(segment
 		(start 141.85 81.5)
 		(end 140.55 80.2)
@@
 	)
 	(segment
+		(start 141.9 79.9)
+		(end 145.3 76.5)
+		(width 0.2)
+		(layer "F.Cu")
+		(net 32)
+	)
+	(segment
 		(start 140.55 80.2)
 		(end 137 80.2)
@@
 	)
 	(segment
-		(start 141.85 81.3)
-		(end 141.85 79.95)
+		(start 145.3 76.5)
+		(end 145.3 75.3)
 		(width 0.2)
 		(layer "F.Cu")
@@
 	)
 	(via
-		(at 145 76.8)
+		(at 145.3 75.3)
 		(size 0.6)
 		(drill 0.3)
@@
 	)
 	(segment
-		(start 146.24 76.8)
-		(end 145 76.8)
-		(width 0.2)
-		(layer "B.Cu")
-		(net 32)
-	)
-	(segment
 		(start 131.5 93.2375)
 		(end 131.5 91.05)
+		(width 0.2)
+		(layer "B.Cu")
+		(net 32)
+	)
+	(segment
+		(start 147.7 75.34)
+		(end 145.34 75.34)
 		(width 0.2)
 		(layer "B.Cu")
@@
 	)
 	(segment
-		(start 147.7 75.34)
-		(end 146.24 76.8)
-		(width 0.2)
-		(layer "B.Cu")
+		(start 145.34 75.34)
+		(end 145.3 75.3)
+		(width 0.2)
+		(layer "B.Cu")
