File: MCU.kicad_sch (KiCad schematic)
At the start: 18 parts, among them U2 STM32F070F6Px

Commit message: generated drill and gerber files, updeted a few datasheets
Changed lines of the file:
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@@
-	(wire
-		(pts
-			(xy 38.1 156.21) (xy 38.1 154.94)
-		)
-		(stroke
-			(width 0)
-			(type default)
-		)
-	)
 	(wire
 		(pts
@@
 	(wire
 		(pts
-			(xy 48.26 156.21) (xy 38.1 156.21)
+			(xy 48.26 156.21) (xy 33.02 156.21)
 		)
 		(stroke
@@
 	(symbol
 		(lib_id "power:GND")
-		(at 38.1 154.94 180)
+		(at 33.02 156.21 0)
 		(unit 1)
 		(exclude_from_sim no)
@@
 		(dnp no)
 		(property "Reference" "#PWR03"
-			(at 38.1 148.59 0)
+			(at 33.02 162.56 0)
 			(effects
 				(font
@@
 		)
 		(property "Value" "GND"
-			(at 35.56 151.384 0)
+			(at 35.56 159.766 0)
 			(effects
 				(font
@@
 		)
 		(property "Footprint" ""
-			(at 38.1 154.94 0)
+			(at 33.02 156.21 0)
 			(effects
 				(font
@@
 		)
 		(property "Datasheet" ""
-			(at 38.1 154.94 0)
+			(at 33.02 156.21 0)
 			(effects
 				(font
@@
 		)
 		(property "Description" "Power symbol creates a global label with name \"GND\" , ground"
-			(at 38.1 154.94 0)
-			(effects
-				(font
+			(at 33.02 156.21 0)
+			(effects
+				(font
