File: PSU.kicad_sch (KiCad schematic)
At the start: 14 parts, among them J5 2 Pin JST, Q1 PMOS, U3 MCP1824S, U4 MCP73113

Commit message: changed power supply of USB to UART to match datasheet, added changes to pcb Signed-off-by: Fozface <tyler.hickling99@gmail.com>
Parts:
- D4: value D_Schottky -> V1FM10-M3/H
- Q1: footprint MyLib:SOT-23 -> MyLib:SOT-23-3
- R8: footprint LED_SMD:LED_1206_3216Metric_Pad1.42x1.75mm_HandSolder -> Resistor_SMD:R_1206_3216Metric_Pad1.30x1.75mm_HandSolder
Changed lines of the file:
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@@
 			)
 		)
-		(property "Footprint" "MyLib:SOT-23"
+		(property "Footprint" "MyLib:SOT-23-3"
 			(at 179.07 87.63 0)
 			(effects
@@
 			)
 		)
-		(property "Datasheet" "https://ngspice.sourceforge.io/docs/ngspice-html-manual/manual.xhtml#cha_MOSFETs"
+		(property "Datasheet" "https://www.infineon.com/assets/row/public/documents/24/49/infineon-bsr315p-ds-en.pdf?fileId=db3a304412b407950112b42acc6143f0"
 			(at 173.99 102.87 0)
 			(effects
@@
 			)
 		)
-		(property "Footprint" "LED_SMD:LED_1206_3216Metric_Pad1.42x1.75mm_HandSolder"
+		(property "Footprint" "Resistor_SMD:R_1206_3216Metric_Pad1.30x1.75mm_HandSolder"
 			(at 155.194 90.424 90)
 			(effects
@@
 			)
 		)
-		(property "Datasheet" ""
+		(property "Datasheet" "https://www.we-online.com/components/products/datasheet/450405020524.pdf"
 			(at 195.58 86.36 0)
 			(effects
@@
 			)
 		)
-		(property "Value" "D_Schottky"
+		(property "Value" "V1FM10-M3/H"
 			(at 173.99 98.7426 90)
 			(effects
@@
 			)
 		)
-		(property "Datasheet" "~"
+		(property "Datasheet" "https://www.vishay.com/docs/87557/v1fm10.pdf"
 			(at 176.53 100.33 0)
 			(effects
